Commit message: bugfix

File: env/model/ohmni.urdf (robot description, URDF)
Before this commit: robot ohmni, 7 links, 6 joints
Links:
- link caster_link: mass 0.12725 -> 5.5

Commit message: bugfix

File: env/model/ohmni.urdf (robot description, URDF)
Before this commit: robot ohmni, 7 links, 6 joints
Links:
- link caster_link: mass 5.5 -> 2.5

Commit message: bugfix

File: env/model/ohmni.urdf (robot description, URDF)
Before this commit: robot ohmni, 7 links, 6 joints
Links:
- link caster_link: mass 2.5 -> 4.5
